Commit message: urdf update

File: urdf/my_bot.urdf (robot description, URDF)
Before this commit: robot my_bot, 7 links, 6 joints
Links:
- removed link left_link_1
- removed link left_link_2
- removed link left_link_3
- removed link right_link_1
- removed link right_link_2
- removed link right_link_3
- added link left1Link1, mass 1; collision cylinder length=0.05 radius=0.012; visual cylinder length=0.05 radius=0.012
- added link left1Link2, mass 2; collision cylinder length=0.12 radius=0.005; visual cylinder length=0.12 radius=0.005
- added link left1Link3, mass 1; collision cylinder length=0.12 radius=0.005; visual cylinder length=0.12 radius=0.005
- added link left2Link1, mass 1; collision cylinder length=0.05 radius=0.012; visual cylinder length=0.05 radius=0.012
- added link left2Link2, mass 2; collision cylinder length=0.12 radius=0.005; visual cylinder length=0.12 radius=0.005
- added link left2Link3, mass 1; collision cylinder length=0.12 radius=0.005; visual cylinder length=0.12 radius=0.005
- added link right1Link1, mass 1; collision cylinder length=0.05 radius=0.012; visual cylinder length=0.05 radius=0.012
- added link right1Link2, mass 2; collision cylinder length=0.12 radius=0.005; visual cylinder length=0.12 radius=0.005
- added link right1Link3, mass 1; collision cylinder length=0.12 radius=0.005; visual cylinder length=0.12 radius=0.005
- added link right2Link1, mass 1; collision cylinder length=0.05 radius=0.012; visual cylinder length=0.05 radius=0.012
- added link right2Link2, mass 2; collision cylinder length=0.12 radius=0.005; visual cylinder length=0.12 radius=0.005
- added link right2Link3, mass 1; collision cylinder length=0.12 radius=0.005; visual cylinder length=0.12 radius=0.005
- link body: geometry collision box size=0.2 0.15 0.015; visual box size=0.2 0.15 0.015
Joints:
- removed joint joint_b_l1
- removed joint joint_b_r1
- removed joint joint_l1_l2
- removed joint joint_l2_l3
- removed joint joint_r1_r2
- removed joint joint_r2_r3
- added joint body_left1Link1: type revolute, parent body, child left1Link1, origin xyz=0.0725 0.0675 0, axis 1 0 0, limit lower=-3.14 upper=6.24 effort=300 velocity=1
- added joint body_left2Link1: type revolute, parent body, child left2Link1, origin xyz=-0.0725 0.0675 0, axis 1 0 0, limit lower=-3.14 upper=6.24 effort=300 velocity=1
- added joint body_right1Link1: type revolute, parent body, child right1Link1, origin xyz=0.0725 -0.0675 0, axis -1 0 0, limit lower=-3.14 upper=6.24 effort=300 velocity=1
- added joint body_right2Link1: type revolute, parent body, child right2Link1, origin xyz=-0.0725 -0.0675 0, axis -1 0 0, limit lower=-3.14 upper=6.24 effort=300 velocity=1
- added joint left1Link1_left1Link2: type revolute, parent left1Link1, child left1Link2, origin xyz=0 0 0.025, axis 0 0 1, limit lower=-1.57 upper=1.57 effort=300 velocity=1
- added joint left1Link2_left1Link3: type revolute, parent left1Link2, child left1Link3, origin xyz=0 0.12 0, axis -0.707 0 0.707, limit lower=-1.57 upper=1.57 effort=300 velocity=0.005
- added joint left2Link1_left2Link2: type revolute, parent left2Link1, child left2Link2, origin xyz=0 0 0.025, axis 0 0 1, limit lower=-1.57 upper=1.57 effort=300 velocity=1
- added joint left2Link2_left2Link3: type revolute, parent left2Link2, child left2Link3, origin xyz=0 0.12 0, axis -0.707 0 0.707, limit lower=-1.57 upper=1.57 effort=300 velocity=0.005
- added joint right1Link1_right1Link2: type revolute, parent right1Link1, child right1Link2, origin xyz=0 0 0.025, axis 0 0 -1, limit lower=-1.57 upper=1.57 effort=300 velocity=1
- added joint right1Link2_right1Link3: type revolute, parent right1Link2, child right1Link3, origin xyz=0 -0.12 0, axis 0.707 0 -0.707, limit lower=-1.57 upper=1.57 effort=300 velocity=0.005
- added joint right2Link1_right2Link2: type revolute, parent right2Link1, child right2Link2, origin xyz=0 0 0.025, axis 0 0 -1, limit lower=-1.57 upper=1.57 effort=300 velocity=1
- added joint right2Link2_right2Link3: type revolute, parent right2Link2, child right2Link3, origin xyz=0 -0.12 0, axis 0.707 0 -0.707, limit lower=-1.57 upper=1.57 effort=300 velocity=0.005

Commit message: 要提交的变更： 	新文件：   LeggedRobotsForBullet-master/.gitignore 	新文件：   LeggedRobotsForBullet-master/LICENSE 	新文件：   LeggedRobotsForBullet-master/README.md 	新文件：   LeggedRobotsForBullet-master/quadrupedal/exmple_stand_up.py 	新文件：   LeggedRobotsForBullet-master/quadrupedal/inverse_dynamics.py 	新文件：   LeggedRobotsForBullet-master/quadrupedal/meshes/stl/abduction_link.stl 	新文件：   LeggedRobotsForBullet-master/quadrupedal/meshes/stl/base.stl 	新文件：   LeggedRobotsForBullet-master/quadrupedal/meshes/stl/lower_link.stl 	新文件：   LeggedRobotsForBullet-master/quadrupedal/meshes/stl/upper_link.stl 	新文件：   LeggedRobotsForBullet-master/quadrupedal/robot.py 	新文件：   LeggedRobotsForBullet-master/quadrupedal/tform.py 	新文件：   LeggedRobotsForBullet-master/quadrupedal/urdf/expansion.sh 	新文件：   LeggedRobotsForBullet-master/quadrupedal/urdf/quadrupedal.urdf 	新文件：   LeggedRobotsForBullet-master/quadrupedal/urdf/quadrupedal.xacro 	修改：     scripts/pybullet_my_bot.py 	删除：     urdf/bennett_bot.urdf 	新文件：   urdf/bennett_linkage.urdf 	新文件：   urdf/my_bot.gv 	新文件：   urdf/my_bot.pdf 	修改：     urdf/my_bot.urdf

File: urdf/my_bot.urdf (robot description, URDF)
Before this commit: robot my_bot, 13 links, 12 joints
Links:
- link body: mass 6 -> 10
